File: switchotron-mems-driver/switchotron-mems-driver-v1.brd (EAGLE design)
At the start: 63.5 x 53.3 mm, 3 parts

Commit message: mems driver design work
Parts:
- added H1, H2: MOUNT-HOLE3.2, holes:3,2
- added J1: 2301841-2, 2301841-2:TE_2301841-2
- moved H4 25.0 mm to (69.8, 69.8)
- moved J3 22.5 mm to (26.7, 73.0)
- moved H3 21.6 mm to (6.35, 69.8)
Other:
- board size 63.5 x 53.3 mm -> 76.2 x 76.2 mm
- board text removed: "2""
Changed lines of the file:
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@@
 <board>
 <plain>
-<wire x1="0" y1="0" x2="63.5" y2="0" width="0.2032" layer="20"/>
-<wire x1="63.5" y1="0" x2="63.5" y2="53.34" width="0.2032" layer="20"/>
-<wire x1="63.5" y1="53.34" x2="0" y2="53.34" width="0.2032" layer="20"/>
-<wire x1="0" y1="53.34" x2="0" y2="0" width="0.2032" layer="20"/>
+<wire x1="0" y1="0" x2="76.2" y2="0" width="0.2032" layer="20"/>
+<wire x1="76.2" y1="0" x2="76.2" y2="76.2" width="0.2032" layer="20"/>
+<wire x1="76.2" y1="76.2" x2="0" y2="76.2" width="0.2032" layer="20"/>
+<wire x1="0" y1="76.2" x2="0" y2="0" width="0.2032" layer="20"/>
 <wire x1="15.494" y1="0.508" x2="15.494" y2="29.21" width="0.0762" layer="51"/>
 <text x="-7.62" y="-5.08" size="2.286" layer="27">Arduino Wee v1.3</text>
 <text x="2.54" y="-2.54" size="1.778" layer="27">Tent Vias!</text>
-<text x="43.815" y="45.72" size="1.27" layer="21" rot="R90">GND</text>
-<text x="26.035" y="46.99" size="1.27" layer="21" rot="R90">D5</text>
-<text x="23.495" y="46.99" size="1.27" layer="21" rot="R90">D4</text>
-<text x="20.955" y="46.99" size="1.27" layer="21" rot="R90">D3</text>
-<text x="33.02" y="43.815" size="2.54" layer="21" rot="R180">2"</text>
-<wire x1="33.655" y1="42.545" x2="57.15" y2="42.545" width="0.254" layer="21"/>
-<wire x1="57.15" y1="42.545" x2="56.515" y2="41.91" width="0.254" layer="21"/>
-<wire x1="57.15" y1="42.545" x2="56.515" y2="43.18" width="0.254" layer="21"/>
-<wire x1="57.15" y1="44.45" x2="57.15" y2="41.91" width="0.254" layer="21"/>
-<wire x1="29.21" y1="42.545" x2="6.35" y2="42.545" width="0.254" layer="21"/>
-<wire x1="6.35" y1="42.545" x2="6.985" y2="43.18" width="0.254" layer="21"/>
-<wire x1="6.35" y1="42.545" x2="6.985" y2="41.91" width="0.254" layer="21"/>
-<wire x1="6.35" y1="41.91" x2="6.35" y2="44.45" width="0.254" layer="21"/>
-<text x="10.16" y="49.53" size="2.54" layer="21">#4</text>
-<text x="59.055" y="50.165" size="2.54" layer="21">#4</text>
-<text x="37.465" y="8.255" size="1.778" layer="21" rot="R180">switchotron-mems-driver-v1
+<text x="50.165" y="67.31" size="1.27" layer="21" rot="R90">GND</text>
+<text x="32.385" y="69.215" size="1.27" layer="21" rot="R90">D5</text>
+<text x="29.845" y="69.215" size="1.27" layer="21" rot="R90">D4</text>
+<text x="27.305" y="69.215" size="1.27" layer="21" rot="R90">D3</text>
+<text x="71.755" y="64.135" size="2.54" layer="21">#4</text>
+<text x="53.34" y="8.89" size="1.778" layer="21" rot="R180">switchotron-mems-driver-v1
 DEC 2023</text>
-<text x="41.275" y="45.085" size="1.27" layer="21" rot="R90">5VDC</text>
+<text x="47.625" y="66.675" size="1.27" layer="21" rot="R90">5VDC</text>
 </plain>
 <attributes>
@@
 </autorouter>
 <elements>
-<element name="J3" library="SparkFun-Connectors" package="1X10" value="" x="20.32" y="51.435" smashed="yes">
-<attribute name="NAME" x="19.05" y="52.832" size="0.6096" layer="25" font="vector" ratio="20"/>
-<attribute name="PROD_ID" value="CONN-11563" x="20.32" y="51.435" size="1.778" layer="27" display="off"/>
-<attribute name="VALUE" x="19.05" y="49.403" size="0.6096" layer="27" font="vector" ratio="20"/>
-</element>
-<element name="H3" library="holes" library_urn="urn:adsk.eagle:library:237" package="3,2" package3d_urn="urn:adsk.eagle:package:14275/1" value="MOUNT-HOLE3.2" x="6.35" y="48.26" smashed="yes">
-<attribute name="POPULARITY" value="7" x="6.35" y="48.26" size="1.778" layer="27" display="off"/>
-</element>
-<element name="H4" library="holes" library_urn="urn:adsk.eagle:library:237" package="3,2" package3d_urn="urn:adsk.eagle:package:14275/1" value="MOUNT-HOLE3.2" x="57.15" y="48.26" smashed="yes">
-<attribute name="POPULARITY" value="7" x="57.15" y="48.26" size="1.778" layer="27" display="off"/>
+<element name="J3" library="SparkFun-Connectors" package="1X10" value="" x="26.67" y="73.025" smashed="yes">
+<attribute name="NAME" x="25.4" y="74.422" size="0.6096" layer="25" font="vector" ratio="20"/>
+<attribute name="PROD_ID" value="CONN-11563" x="26.67" y="73.025" size="1.778" layer="27" display="off"/>
+<attribute name="VALUE" x="25.4" y="70.993" size="0.6096" layer="27" font="vector" ratio="20"/>
+</element>
+<element name="H3" library="holes" library_urn="urn:adsk.eagle:library:237" package="3,2" package3d_urn="urn:adsk.eagle:package:14275/1" value="MOUNT-HOLE3.2" x="6.35" y="69.85" smashed="yes">
+<attribute name="POPULARITY" value="7" x="6.35" y="69.85" size="1.778" layer="27" display="off"/>
+</element>
+<element name="H4" library="holes" library_urn="urn:adsk.eagle:library:237" package="3,2" package3d_urn="urn:adsk.eagle:package:14275/1" value="MOUNT-HOLE3.2" x="69.85" y="69.85" smashed="yes">
+<attribute name="POPULARITY" value="7" x="69.85" y="69.85" size="1.778" layer="27" display="off"/>
+</element>
+<element name="J1" library="2301841-2" package="TE_2301841-2" value="2301841-2" x="38.1" y="17.145" smashed="yes">
+<attribute name="MANUFACTURER" value="TE Connectivity" x="38.1" y="17.145" size="1.778" layer="27" display="off"/>
+<attribute name="MAXIMUM_PACKAGE_HEIGHT" value="10.90 mm" x="38.1" y="17.145" size="1.778" layer="27" display="off"/>
+<attribute name="NAME" x="11.35" y="23.895" size="1.27" layer="25"/>
+<attribute name="PARTREV" value="E" x="38.1" y="17.145" size="1.778" layer="27" display="off"/>
+<attribute name="STANDARD" value="Manufacturer Recommendation" x="38.1" y="17.145" size="1.778" layer="27" display="off"/>
+<attribute name="VALUE" x="11.35" y="9.145" size="1.27" layer="27"/>
+</element>
+<element name="H1" library="holes" library_urn="urn:adsk.eagle:library:237" package="3,2" package3d_urn="urn:adsk.eagle:package:14275/1" value="MOUNT-HOLE3.2" x="6.35" y="6.35" smashed="yes">
+<attribute name="POPULARITY" value="7" x="6.35" y="6.35" size="1.778" layer="27" display="off"/>
+</element>
+<element name="H2" library="holes" library_urn="urn:adsk.eagle:library:237" package="3,2" package3d_urn="urn:adsk.eagle:package:14275/1" value="MOUNT-HOLE3.2" x="69.85" y="6.35" smashed="yes">
+<attribute name="POPULARITY" value="7" x="69.85" y="6.35" size="1.778" layer="27" display="off"/>
 </element>
 </elements>
@@
 <polygon width="0.254" layer="1" isolate="0.3048">
 <vertex x="-1.905" y="-1.27"/>
-<vertex x="-1.905" y="56.515"/>
-<vertex x="64.135" y="56.515"/>
-<vertex x="64.135" y="-1.27"/>
+<vertex x="-1.905" y="77.47"/>
+<vertex x="78.105" y="77.47"/>
+<vertex x="78.105" y="-1.27"/>
 </polygon>
 <polygon width="0.254" layer="16" isolate="0.3048">
 <vertex x="-3.81" y="-2.54"/>
-<vertex x="-3.81" y="56.515"/>
-<vertex x="65.405" y="56.515"/>
-<vertex x="65.405" y="-2.54"/>
+<vertex x="-3.81" y="79.375"/>
+<vertex x="80.01" y="79.375"/>
+<vertex x="80.01" y="-2.54"/>
 </polygon>
 </signal>
