File: switchotron-mems-driver/switchotron-mems-driver-v1.sch (EAGLE design)
At the start: 3 parts

Commit message: mems driver design work
Parts:
- added H1, H2: MOUNT-HOLE3.2, holes:MOUNT-HOLE3.2
- added J1: 2301841-2, 2301841-2:2301841-2
Changed lines of the file:
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@@
 <part name="H3" library="holes" library_urn="urn:adsk.eagle:library:237" deviceset="MOUNT-HOLE" device="3.2" package3d_urn="urn:adsk.eagle:package:14275/1"/>
 <part name="H4" library="holes" library_urn="urn:adsk.eagle:library:237" deviceset="MOUNT-HOLE" device="3.2" package3d_urn="urn:adsk.eagle:package:14275/1"/>
+<part name="J1" library="2301841-2" deviceset="2301841-2" device=""/>
+<part name="H1" library="holes" library_urn="urn:adsk.eagle:library:237" deviceset="MOUNT-HOLE" device="3.2" package3d_urn="urn:adsk.eagle:package:14275/1"/>
+<part name="H2" library="holes" library_urn="urn:adsk.eagle:library:237" deviceset="MOUNT-HOLE" device="3.2" package3d_urn="urn:adsk.eagle:package:14275/1"/>
 </parts>
 <sheets>
@@
 <attribute name="VALUE" x="163.322" y="127.0762" size="1.778" layer="96"/>
 </instance>
+<instance part="J1" gate="G$1" x="132.08" y="95.25" smashed="yes">
+<attribute name="NAME" x="124.46" y="114.3" size="1.778" layer="95"/>
+<attribute name="VALUE" x="124.46" y="72.39" size="1.778" layer="96"/>
+</instance>
+<instance part="H1" gate="G$1" x="92.71" y="123.19" smashed="yes">
+<attribute name="NAME" x="94.742" y="123.7742" size="1.778" layer="95"/>
+<attribute name="VALUE" x="94.742" y="120.7262" size="1.778" layer="96"/>
+</instance>
+<instance part="H2" gate="G$1" x="161.29" y="120.65" smashed="yes">
+<attribute name="NAME" x="163.322" y="121.2342" size="1.778" layer="95"/>
+<attribute name="VALUE" x="163.322" y="118.1862" size="1.778" layer="96"/>
+</instance>
 </instances>
